Commit message: feat: New alphabot model

File: src/ROS/alphabot2_description/urdf/alphabot2.urdf (robot description, URDF)
Before this commit: robot alphabot2, 3 links, 2 joints
Links:
- removed link link_chassis
- removed link link_left_wheel
- removed link link_right_wheel
- added link base_link; visual cylinder length=0.003 radius=0.055
- added link body; visual box size=0.09 0.06 0.04
- added link casterBallFront; visual sphere radius=0.005
- added link casterBallRear; visual sphere radius=0.005
- added link casterFront; visual cylinder length=0.01 radius=0.005
- added link casterRear; visual cylinder length=0.01 radius=0.005
- added link top; visual cylinder length=0.003 radius=0.055
- added link wheelLeft; visual cylinder length=0.025 radius=0.022
- added link wheelRight; visual cylinder length=0.025 radius=0.022
Joints:
- removed joint joint_left_wheel
- removed joint joint_right_wheel
- added joint body_joint: type fixed, parent base_link, child body, origin xyz=0 0 0.0215 rpy=0 0 0
- added joint casterBallFront_joint: type fixed, parent casterFront, child casterBallFront, origin xyz=0.0 0.0 -0.003 rpy=0 0 0
- added joint casterBallRear_joint: type fixed, parent casterRear, child casterBallRear, origin xyz=0.0 0.0 -0.003 rpy=0 0 0
- added joint casterFront_joint: type fixed, parent base_link, child casterFront, origin xyz=0.05 0.0 -0.0065 rpy=0 0 0
- added joint casterRear_joint: type fixed, parent base_link, child casterRear, origin xyz=-0.05 0.0 -0.0065 rpy=0 0 0
- added joint top_joint: type fixed, parent body, child top, origin xyz=0 0 0.0215 rpy=0 0 0
- added joint wheelLeft_joint: type continuous, parent base_link, child wheelLeft, origin xyz=0.0 0.04 0.007 rpy=0 0 0, axis 0 1 0, limit effort=10000 velocity=1000
- added joint wheelRight_joint: type continuous, parent base_link, child wheelRight, origin xyz=0.0 -0.04 0.007 rpy=0 0 0, axis 0 1 0, limit effort=10000 velocity=1000

Commit message: feat: Working model

File: src/ROS/alphabot2_description/urdf/alphabot2.urdf (robot description, URDF)
Before this commit: robot alphabot2, 9 links, 8 joints
Links:
- removed link base_link
- removed link top
- added link bottom_plate, mass 0.5; collision cylinder length=0.003 radius=0.055; visual cylinder length=0.003 radius=0.055
- added link top_plate, mass 0.05; collision cylinder length=0.003 radius=0.055; visual cylinder length=0.003 radius=0.055
- link body: mass None -> 0.3; geometry collision box size=0.09 0.06 0.04; visual box size=0.09 0.06 0.04
- link casterBallFront: mass None -> 0.005; geometry collision sphere radius=0.005; visual sphere radius=0.005
- link casterBallRear: mass None -> 0.005; geometry collision sphere radius=0.005; visual sphere radius=0.005
- link casterFront: mass None -> 0.01; geometry collision cylinder length=0.01 radius=0.005; visual cylinder length=0.01 radius=0.005
- link casterRear: mass None -> 0.01; geometry collision cylinder length=0.01 radius=0.005; visual cylinder length=0.01 radius=0.005
- link wheelLeft: mass None -> 0.02; geometry collision cylinder length=0.025 radius=0.022; visual cylinder length=0.025 radius=0.022
- link wheelRight: mass None -> 0.02; geometry collision cylinder length=0.025 radius=0.022; visual cylinder length=0.025 radius=0.022
Joints:
- joint body_joint: parent base_link -> bottom_plate
- joint casterFront_joint: parent base_link -> bottom_plate
- joint casterRear_joint: parent base_link -> bottom_plate
- joint top_joint: child top -> top_plate
- joint wheelLeft_joint: parent base_link -> bottom_plate
- joint wheelRight_joint: parent base_link -> bottom_plate

Commit message: refactor: Estimated intertial values

File: src/ROS/alphabot2_description/urdf/alphabot2.urdf (robot description, URDF)
Before this commit: robot alphabot2, 9 links, 8 joints
Links:
- link body: mass 0.3 -> 0.26
- link bottom_plate: mass 0.5 -> 0.08
- link casterBallFront: mass 0.005 -> 0.000628
- link casterBallRear: mass 0.005 -> 0.000628
- link casterFront: mass 0.01 -> 0.00094
- link casterRear: mass 0.01 -> 0.00094
- link top_plate: mass 0.05 -> 0.0342
- link wheelLeft: mass 0.02 -> 0.04
- link wheelRight: mass 0.02 -> 0.04
